File: hayashibalab/adrobo/adrobo.kicad_pcb (KiCad board)
At the start: 2 copper layers, 64 parts, among them J1 Batt, J10 Conn_01x05, J11 CN2, J12 CN1, J13 UART2, J14 SWD, J2 ADC, J3 Conn_01x05, J4 Conn_01x05, J5 SERVO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

Commit message: 何をコミットしたのかよくわからん
Parts:
- removed J10, J4, J9: Conn_01x05, Connector_PinHeader_2.54mm:PinHeader_1x05_P2.54mm_Vertical
- removed J5: SERVO, Connector_PinHeader_2.54mm:PinHeader_1x04_P2.54mm_Vertical
- removed J6, J7: Conn_01x04, Connector_PinHeader_2.54mm:PinHeader_1x04_P2.54mm_Vertical
- removed J8: GPIO, Connector_PinHeader_2.54mm:PinHeader_1x05_P2.54mm_Vertical
- added C11: 0.1u, Capacitor_SMD:C_0603_1608Metric, B.Cu at (76.2, 58.0)
- added C12: 0.1u, Capacitor_SMD:C_0603_1608Metric, B.Cu at (74.8, 58.0)
- added C13: 0.1u, Capacitor_SMD:C_0603_1608Metric, B.Cu at (79.2, 58.0)
- added C14: 0.1u, Capacitor_SMD:C_0603_1608Metric, B.Cu at (77.8, 58.0)
- added C15: 4.7u, Capacitor_SMD:C_0603_1608Metric, B.Cu at (80.8, 58.0)
- added C7: 0.1u, Capacitor_SMD:C_0603_1608Metric, F.Cu at (113.8, 83.0)
- added C8: 0.1u, Capacitor_SMD:C_0603_1608Metric, B.Cu at (102.2, 83.5)
- added G***: LOGO, logo:soiya, B.Cu at (111.8, 46.8)
- added REF**: MountingHole_3.2mm_M3_Pad, MountingHole:MountingHole_3.2mm_M3_Pad, F.Cu at (127.5, 95.0)
- added REF**: MountingHole_3.2mm_M3_Pad, MountingHole:MountingHole_3.2mm_M3_Pad, F.Cu at (65.5, 48.5)
- added REF**: MountingHole_3.2mm_M3_Pad, MountingHole:MountingHole_3.2mm_M3_Pad, F.Cu at (65.5, 95.0)
- added REF**: MountingHole_3.2mm_M3_Pad, MountingHole:MountingHole_3.2mm_M3_Pad, F.Cu at (127.5, 48.5)
- added U5: NJU7223DL1, original:Regulator, B.Cu at (107.2, 83.0)
- added U6: SERVO, original:PinHeader_3x04_P2.54mm_Vertical, B.Cu at (108.8, 93.5)
- C1, C4, C5, C6, D18, D19, R12, R14, U1: moved to B.Cu
- J2: footprint Connector_PinHeader_2.54mm:PinHeader_1x05_P2.54mm_Vertical -> original:PinHeader_3x05_P2.54mm_Vertical; moved to B.Cu
- J3: value Conn_01x05 -> GPIO; footprint Connector_PinHeader_2.54mm:PinHeader_1x05_P2.54mm_Vertical -> original:PinHeader_3x05_P2.54mm_Vertical
- moved C2 90.6 mm to (121.8, 83.2), turned to 90 degrees
- moved U3 86.5 mm to (108.8, 62.0), turned to 180 degrees
- moved J11 86.2 mm to (127.2, 65.5)
- moved U2 83.0 mm to (80.2, 85.5), turned to 270 degrees
- moved C1 82.8 mm to (124.2, 83.2), turned to 90 degrees
- moved J3 76.6 mm to (79.8, 93.5), turned to 180 degrees
- moved J2 74.8 mm to (94.8, 93.5)
- moved J12 69.8 mm to (127.2, 55.5)
- moved D14 67.4 mm to (124.8, 72.5), turned to 270 degrees
- moved D18 66.9 mm to (124.8, 64.0), turned to 270 degrees
- moved D17 66.3 mm to (121.8, 52.5), turned to 270 degrees
- moved D15 63.2 mm to (121.8, 72.5), turned to 270 degrees
- moved D16 59.9 mm to (118.8, 52.5), turned to 270 degrees
- moved D12 55.9 mm to (124.0, 61.0), turned to 270 degrees
- moved D19 55.7 mm to (121.8, 64.0), turned to 270 degrees
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Connections:
- C1 pad 1: Net-(C1-Pad1) -> +9V
- C2 pad 1: +5V -> +9V
- C4 pad 1: Net-(C4-Pad1) -> +9V
- D1 pad 2: PA7 -> PA0
- D11 pad 1: Net-(D11-Pad1) -> +9V
- D11 pad 2: /OUT2 -> /MOTOROUT2
- D12 pad 1: Net-(D11-Pad1) -> +9V
- D12 pad 2: /OUT1 -> /MOTOROUT1
- D14 pad 1: /OUT2 -> /MOTOROUT2
- D15 pad 1: /OUT1 -> /MOTOROUT1
- D16 pad 1: Net-(D16-Pad1) -> +9V
- D16 pad 2: /OUT4 -> /MOTOROUT4
- D17 pad 1: Net-(D16-Pad1) -> +9V
- D17 pad 2: /OUT3 -> /MOTOROUT3
- D18 pad 1: /OUT4 -> /MOTOROUT4
- D19 pad 1: /OUT3 -> /MOTOROUT3
- D2 pad 2: PA6 -> PA4
- D4 pad 2: PA4 -> PA6
- D5 pad 2: PA0 -> PA7
- J1 pad 2: Net-(C1-Pad1) -> +9V
- J11 pad 1: /OUT1 -> /MOTOROUT1
- J11 pad 2: /OUT2 -> /MOTOROUT2
- J12 pad 1: /OUT3 -> /MOTOROUT3
- J12 pad 2: /OUT4 -> /MOTOROUT4
- J3 pad 1: +5V -> PA12
- J3 pad 2: +5V -> PB7
- J3 pad 3: +5V -> PB6
- J3 pad 4: +5V -> PF0
- J3 pad 5: +5V -> PF1
- R1 pad 2: PA7 -> PA0
- R2 pad 2: PA6 -> PA4
- R4 pad 2: PA4 -> PA6
- R5 pad 2: PA0 -> PA7
- R7 pad 1: (no net) -> +9V
- U1 pad 1: Net-(C1-Pad1) -> +9V
- U3 pad 10: GND -> +9V
- U3 pad 13: /OUT3 -> /MOTOROUT3
- U3 pad 18: /OUT4 -> /MOTOROUT4
- U3 pad 20: Net-(C4-Pad1) -> +9V
- U3 pad 3: /OUT1 -> /MOTOROUT1
- U3 pad 8: /OUT2 -> /MOTOROUT2
Routing:
- net +3V3: track 0.00 -> 150.5 mm, vias 0 -> 10
- net +5V: track 0.00 -> 144.0 mm, vias 0 -> 4
- net +9V: track 0.00 -> 116.1 mm
- net PB6: track 0.00 -> 85.9 mm
- net PF0: track 0.00 -> 73.0 mm, vias 0 -> 2
- net Net-(J14-Pad4): track 0.00 -> 70.8 mm, vias 0 -> 2
- net PF1: track 0.00 -> 65.4 mm, vias 0 -> 2
- net /MOTOROUT4: track 0.00 -> 56.1 mm, vias 0 -> 2
- net Net-(J13-Pad2): track 0.00 -> 54.5 mm, vias 0 -> 5
- net PB7: track 0.00 -> 54.1 mm, vias 0 -> 3
- net PA12: track 0.00 -> 52.4 mm, vias 0 -> 5
- net /MOTOROUT3: track 0.00 -> 52.0 mm, vias 0 -> 2
- net PA11: track 0.00 -> 42.1 mm
- net PA10: track 0.00 -> 40.9 mm
- net PWM: track 0.00 -> 40.8 mm, vias 0 -> 6
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- added copper zone on B.Cu, net GND
- added copper zone on F.Cu, net GND
Other:
- board outline added: 72 x 56.5 mm
- board text added: "1 2 3 4"
- board text added: "1 2 3 4 5"
- board text added: "1 2 3 4 5 6"
- board text added: "ADC"
- board text added: "CN1"
- board text added: "CN2"
- board text added: "GND"
- board text added: "GPIO"
- board text added: "POWER"
- board text added: "SERVO"
- board text added: "SIG"
- board text added: "SW1"
- board text added: "SW2"
- board text added: "SWD"
- board text added: "UART"
- board text added: "V+"
