File: hayashibalab/adrobo/adrobo.sch (KiCad schematic (older format))
At the start: 64 parts, among them J1 Batt, J10 Conn_01x05, J11 CN2, J12 CN1, J13 UART2, J14 SWD, J2 ADC, J3 Conn_01x05, J4 Conn_01x05, J5 SERVO, J6 Conn_01x04, J7 Conn_01x04, J8 GPIO, J9 Conn_01x05, SW1 Switch, SW2 Switch, SW3 Switch, U1 NJM7805SDL1, U2 SN74HC04PWR, U3 L293E, U4 STM32F303K8Tx

Commit message: 何をコミットしたのかよくわからん
Parts:
- removed J10, J3, J4, J9: Conn_01x05, Connector_PinHeader_2.54mm:PinHeader_1x05_P2.54mm_Vertical, symbol Connector_Generic:Conn_01x05
- removed J2: ADC, Connector_PinHeader_2.54mm:PinHeader_1x05_P2.54mm_Vertical, symbol Connector_Generic:Conn_01x05
- removed J5: SERVO, Connector_PinHeader_2.54mm:PinHeader_1x04_P2.54mm_Vertical, symbol Connector_Generic:Conn_01x04
- removed J6, J7: Conn_01x04, Connector_PinHeader_2.54mm:PinHeader_1x04_P2.54mm_Vertical, symbol Connector_Generic:Conn_01x04
- removed J8: GPIO, Connector_PinHeader_2.54mm:PinHeader_1x05_P2.54mm_Vertical, symbol Connector_Generic:Conn_01x05
- added C11, C12, C13, C14, C7, C8: 0.1u, Capacitor_SMD:C_0603_1608Metric, symbol Device:C
- added C15: 4.7u, Capacitor_SMD:C_0603_1608Metric, symbol Device:C
- added J2: ADC, original:PinHeader_3x05_P2.54mm_Vertical, symbol original:Conn_03x_05_Male
- added J3: GPIO, original:PinHeader_3x05_P2.54mm_Vertical, symbol original:Conn_03x_05_Male
- added U5: NJU7223DL1, original:Regulator, symbol original:Regulator
- added U6: SERVO, original:PinHeader_3x04_P2.54mm_Vertical, symbol original:Conn_03x04_Male
Connections:
- net +3V3: now also C11.1, C12.1, C13.1, C14.1, C15.1, C8.1, U5.3 (OUT)
- net +5V: now also C7.1, J2.10, J2.6, J2.7, J2.8, J2.9, J3.10, J3.6, J3.7, J3.8, J3.9, U5.1 (IN), U6.5, U6.6, U6.7, U6.8; no longer C2.1
- net GND: now also C11.2, C12.2, C13.2, C14.2, C15.2, C7.2, C8.2, J2.11, J2.12, J2.13, J2.14, J2.15, J3.11, J3.12, J3.13, J3.14, J3.15, U5.2 (GND), U6.10, U6.11, U6.12, U6.9; no longer U3.10 (VS)
- net OUT1: no longer D12.2 (A), D15.1 (K), J11.1 (Pin_1), U3.3 (OUTPUT_1)
- net OUT2: no longer D11.2 (A), D14.1 (K), J11.2 (Pin_2), U3.8 (OUTPUT_2)
- net OUT3: no longer D17.2 (A), D19.1 (K), J12.1 (Pin_1), U3.13 (OUTPUT_3)
- net OUT4: no longer D16.2 (A), D18.1 (K), J12.2 (Pin_2), U3.18 (OUTPUT_4)
- net PA0: now also D1.2 (A), R1.2; no longer D5.2 (A), R5.2
- net PA10: now also U6.3
- net PA11: now also U6.4
- net PA12: now also J3.1
- net PA4: now also D2.2 (A), R2.2; no longer D4.2 (A), R4.2
- net PA6: now also D4.2 (A), R4.2; no longer D2.2 (A), R2.2
- net PA7: now also D5.2 (A), R5.2; no longer D1.2 (A), R1.2
- net PA8: now also U6.1
- net PA9: now also U6.2
- net PB6: now also J3.3
- net PB7: now also J3.2
- net PF0: now also J3.4
- net PF1: now also J3.5
- net +9V: now reaches C1.1, J1.2 (Pin_2), U1.1 (IN)
- net +9V: now also C2.1, C4.1, D11.1 (K), D12.1 (K), D16.1 (K), D17.1 (K), R7.1, U3.10 (VS), U3.20 (VSS)
- net at R1.1: now also J2.1
- net at R2.1: now also J2.2
- net at R3.1: now also J2.3
- net at R4.1: now also J2.4
- net at R5.1: now also J2.5
- new net MOTOROUT1: D12.2 (A), D15.1 (K), J11.1 (Pin_1), U3.3 (OUTPUT_1)
- new net MOTOROUT2: D11.2 (A), D14.1 (K), J11.2 (Pin_2), U3.8 (OUTPUT_2)
- new net MOTOROUT3: D17.2 (A), D19.1 (K), J12.1 (Pin_1), U3.13 (OUTPUT_3)
- new net MOTOROUT4: D16.2 (A), D18.1 (K), J12.2 (Pin_2), U3.18 (OUTPUT_4)
Other:
- moved on the sheet: C2, U1
